File: Schematics/toadstool mega328.sch (KiCad schematic (older format))
At the start: 25 parts, among them CON1 BARREL_JACK, IC1 ATMEGA328P-P, K1 SHIELD, K2 V-SELECT, K4 ICSP, K5 PIN 2-8, K6 PIN 21-28, K7 XTAL, K8 PIN 15-19, K9 PIN 11-14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

Commit message: Components Changed
Updated Power Jack and Reset button with 3D models.
Minor changes to silkscreen
Parts:
- K4: footprint Pin_Headers:Pin_Header_Straight_2x03 -> Toadstool:ICSP_Header_2x03
Changed lines of the file:
@@
 F 0 "K4" H 8200 3350 50  0000 C CNN
 F 1 "ICSP" H 8200 2950 50  0000 C CNN
-F 2 "Pin_Headers:Pin_Header_Straight_2x03" H 8200 1950 60  0001 C CNN
+F 2 "Toadstool:ICSP_Header_2x03" H 8200 1950 60  0001 C CNN
 F 3 "" H 8200 1950 60  0000 C CNN
 	1    8200 3150
